File: batteryboard-v01c/batteryboard.kicad_pcb (KiCad board)
At the start: 4 copper layers, 95.9 x 90.2 mm, 83 parts, among them J1 KEYSTONE-1042, J2 KEYSTONE-1042, J3 KEYSTONE-1042, J4 KEYSTONE-1042, J5 KEYSTONE-1042, J6 KEYSTONE-1042, J7 Molex 5023521200, J8 Screw_Terminal_01x02, J9 Molex 5023520600, Q1 IRF7458, Q10 IRLML2803, Q11 IRF7404TRPBF, Q2 IRF7458, Q3 IRLML2803, Q4 CSD17579Q5A, Q5 CSD17579Q5A, Q6 BSS138DWQ-7, Q7 MBT2222ADW1T1, Q8 BSS138DWQ-7, Q9 MBT2222ADW1T1, U1 R5460N233AF, U2 BQ28Z620

Commit message: Optimized coil shape
Routing:
- net PACK-: track 909.5 -> 901.8 mm
